File: Board/TATransmitter.kicad_sch (KiCad schematic)
At the start: 11 parts, among them J1 Screw_Terminal_01x03, U1 ESP32-DevKitC, U2 ADS1115IDGS

Commit message: R6 von 2K auf 5k geändert entspricht TA = 2.0
Parts:
- R6: value 2k -> 5k
Changed lines of the file:
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@@
     (pin "1")
     (instances
-      (project "ESP32"
+      (project "TATransmitter"
         (path "/6bca0369-8be4-4b0a-98a0-8352f7b9aa16"
           (reference "R7") (unit 1)
@@
     (pin "1")
     (instances
-      (project "ESP32"
+      (project "TATransmitter"
         (path "/6bca0369-8be4-4b0a-98a0-8352f7b9aa16"
           (reference "#PWR011") (unit 1)
@@
     (pin "1")
     (instances
-      (project "ESP32"
+      (project "TATransmitter"
         (path "/6bca0369-8be4-4b0a-98a0-8352f7b9aa16"
           (reference "R3") (unit 1)
@@
     (pin "1")
     (instances
-      (project "ESP32"
+      (project "TATransmitter"
         (path "/6bca0369-8be4-4b0a-98a0-8352f7b9aa16"
           (reference "#PWR08") (unit 1)
@@
       (effects (font (size 1.27 1.27)) (justify left))
     )
-    (property "Value" "2k" (at 165.1 48.26 0)
+    (property "Value" "5k" (at 165.1 48.26 0)
       (effects (font (size 1.27 1.27)) (justify left))
     )
@@
     (pin "1")
     (instances
-      (project "ESP32"
+      (project "TATransmitter"
         (path "/6bca0369-8be4-4b0a-98a0-8352f7b9aa16"
           (reference "R6") (unit 1)
@@
     (pin "21")
     (instances
-      (project "ESP32"
+      (project "TATransmitter"
         (path "/6bca0369-8be4-4b0a-98a0-8352f7b9aa16"
           (reference "U1") (unit 1)
@@
     (pin "2")
     (instances
-      (project "ESP32"
+      (project "TATransmitter"
         (path "/6bca0369-8be4-4b0a-98a0-8352f7b9aa16"
           (reference "R4") (unit 1)
@@
     (pin "1")
     (instances
-      (project "ESP32"
+      (project "TATransmitter"
         (path "/6bca0369-8be4-4b0a-98a0-8352f7b9aa16"
           (reference "R1") (unit 1)
@@
     (pin "1")
     (instances
-      (project "ESP32"
+      (project "TATransmitter"
         (path "/6bca0369-8be4-4b0a-98a0-8352f7b9aa16"
           (reference "#PWR01") (unit 1)
@@
     (pin "1")
     (instances
-      (project "ESP32"
+      (project "TATransmitter"
         (path "/6bca0369-8be4-4b0a-98a0-8352f7b9aa16"
           (reference "R5") (unit 1)
@@
     (pin "1")
     (instances
-      (project "ESP32"
+      (project "TATransmitter"
         (path "/6bca0369-8be4-4b0a-98a0-8352f7b9aa16"
           (reference "#PWR05") (unit 1)
@@
     (pin "1")
     (instances
-      (project "ESP32"
+      (project "TATransmitter"
         (path "/6bca0369-8be4-4b0a-98a0-8352f7b9aa16"
           (reference "#PWR03") (unit 1)
@@
     (pin "3")
     (instances
-      (project "ESP32"
+      (project "TATransmitter"
         (path "/6bca0369-8be4-4b0a-98a0-8352f7b9aa16"
           (reference "U2") (unit 1)
@@
     (pin "1")
     (instances
-      (project "ESP32"
+      (project "TATransmitter"
         (path "/6bca0369-8be4-4b0a-98a0-8352f7b9aa16"
           (reference "#PWR07") (unit 1)
@@
     (pin "1")
     (instances
-      (project "ESP32"
+      (project "TATransmitter"
         (path "/6bca0369-8be4-4b0a-98a0-8352f7b9aa16"
           (reference "R2") (unit 1)
@@
     (pin "1")
     (instances
-      (project "ESP32"
+      (project "TATransmitter"
         (path "/6bca0369-8be4-4b0a-98a0-8352f7b9aa16"
           (reference "#PWR09") (unit 1)
@@
     (pin "2")
     (instances
-      (project "ESP32"
+      (project "TATransmitter"
         (path "/6bca0369-8be4-4b0a-98a0-8352f7b9aa16"
           (reference "C1") (unit 1)
@@
     (pin "1")
     (instances
-      (project "ESP32"
+      (project "TATransmitter"
         (path "/6bca0369-8be4-4b0a-98a0-8352f7b9aa16"
           (reference "#PWR04") (unit 1)
@@
     (pin "1")
     (instances
-      (project "ESP32"
+      (project "TATransmitter"
         (path "/6bca0369-8be4-4b0a-98a0-8352f7b9aa16"
           (reference "#PWR06") (unit 1)
@@
     (pin "1")
     (instances
-      (project "ESP32"
+      (project "TATransmitter"
         (path "/6bca0369-8be4-4b0a-98a0-8352f7b9aa16"
           (reference "#PWR02") (unit 1)
@@
     (pin "1")
     (instances
-      (project "ESP32"
+      (project "TATransmitter"
         (path "/6bca0369-8be4-4b0a-98a0-8352f7b9aa16"
           (reference "J1") (unit 1)
